Commit message: Robot base control

File: speedy_description/robots/speedy.urdf.xacro (robot description, xacro)
@@ -118,10 +118,14 @@
                           xyz_offset="0.09844 -0.00000 0.00000"
                           rpy="0.00000 0.00000 0.0000"
-                          robot_ns="$(arg robot_ns)"/>
+                          robot_ns="$(arg robot_ns)"
+                          video_width="640"
+                          video_height="480"/>
     <xacro:sensor_camera  prefix="$(arg prefix)gripper_"
-                          parent_link="$(arg prefix)gripper_camera_link"
-                          xyz_offset="0.000000 -0.00000 0.00000"
+                          parent_link="$(arg prefix)gripper_base_link"
+                          xyz_offset="0.000000 -0.05000 0.0000"
                           rpy="${-PI/2} 0.00000 ${-PI/2}"
-                          robot_ns="$(arg robot_ns)"/>
+                          robot_ns="$(arg robot_ns)"
+                          video_width="640"
+                          video_height="480"/>
     <xacro:sensor_imu prefix="$(arg prefix)base_"
                       parent_link="$(arg prefix)base_link"
@@ -131,8 +135,8 @@
                       topic="base_imu"/>
     <!-- GAZEBO ROS2 CONTROL -->
-    <!--xacro:include filename="$(find speedy_description)/urdf/ros2_control.urdf.xacro"/>
+    <xacro:include filename="$(find speedy_description)/urdf/ros2_control.urdf.xacro"/>
     <xacro:arg name="config_controllers" default="$(find speedy_description)/config/speedy_controllers.yaml"/>
     <xacro:arg name="update_rate" default="20"/>
-    <xacro:ros2_control/-->
+    <xacro:ros2_control frame_prefix="$(arg prefix)"/>
     <!-- MATERIALS -->
     <material name="Material">

File: speedy_description/urdf/arm/gripper.urdf.xacro (robot description, xacro)
@@ -101,10 +101,4 @@
                                 material="${white_material}"
                                 prefix="${prefix}"/>
-    <link name="${prefix}gripper_camera_link"/>
-    <joint name="${prefix}gripper_camera_link_joint" type="fixed">
-        <origin rpy="-1.57080 -0.00000 -1.57080" xyz="0.00000 -0.05000 0.00000"/>
-        <parent link="${prefix}gripper_base_link"/>
-        <child link="${prefix}gripper_camera_link"/>
-    </joint>
     </xacro:macro>
 </robot>

File: speedy_description/urdf/base/robot_base.urdf.xacro (robot description, xacro)
@@ -131,5 +131,5 @@
     <link name="${prefix}camera_2_link">
       <collision name="camera_2_collision">
-        <origin rpy="0.00000 0.00000 0.00000" xyz="0.00000 0.00000 0.00000"/>
+        <origin rpy="0.00000 ${PI/2} 0.00000" xyz="0.00000 0.00000 0.00000"/>
         <geometry>
           <mesh filename="file://$(find speedy_description)/meshes/dae/Cylinder.009.dae" scale="1.00000 1.00000 1.00000"/>
@@ -137,5 +137,5 @@
       </collision>
       <visual name="camera_2">
-        <origin rpy="0.00000 -0.00000 0.00000" xyz="0.00000 0.00000 0.00000"/>
+        <origin rpy="0.00000 ${PI/2} 0.00000" xyz="0.00000 0.00000 0.00000"/>
         <material name="Material.007"/>
         <geometry>
@@ -149,5 +149,19 @@
       <child link="${prefix}camera_2_link"/>
     </joint>
-    <link name="${prefix}front_camera_lens_link"/>
+    <link name="${prefix}front_camera_lens_link">
+      <collision name="camera_collision">
+        <origin rpy="0.00000 ${PI/2} 0.00000" xyz="0.00000 -0.00000 -0.00000"/>
+        <geometry>
+          <cylinder radius="0.0764605" length="0.02"/>
+        </geometry>
+      </collision>
+      <visual name="camera">
+        <origin rpy="0.00000 ${PI/2} 0.00000" xyz="0.00000 0.00000 -0.00000"/>
+        <material name="grey"/>
+        <geometry>
+          <cylinder radius="0.0764605" length="0.02"/>
+        </geometry>
+      </visual>
+    </link>
     <joint name="${prefix}camera_lens_link_joint" type="fixed">
       <origin rpy="-0.00000 0.000 0.00000" xyz="0.36378 -0.09634 0.02978"/>
@@ -157,5 +171,5 @@
     <link name="${prefix}front_camera_objective_link">
       <collision name="camera_collision">
-        <origin rpy="0.00000 0.00000 0.00000" xyz="0.00000 -0.00000 -0.00000"/>
+        <origin rpy="0.00000 ${PI/2} 0.00000" xyz="0.00000 -0.00000 -0.00000"/>
         <geometry>
           <mesh filename="file://$(find speedy_description)/meshes/dae/Cylinder.004.dae" scale="0.35487 0.35487 0.44358"/>
@@ -163,5 +177,5 @@
       </collision>
       <visual name="camera">
-        <origin rpy="0.00000 -0.00000 0.00000" xyz="0.00000 0.00000 -0.00000"/>
+        <origin rpy="0.00000 ${PI/2} 0.00000" xyz="0.00000 0.00000 -0.00000"/>
         <material name="Material.005"/>
         <geometry>
@@ -177,5 +191,5 @@
     <link name="${prefix}head_link">
       <collision name="head_collision">
-        <origin rpy="0.00000 0.00000 0.00000" xyz="0.00000 0.00016 -0.00000"/>
+        <origin rpy="0.00000 ${PI/2} 0.00000" xyz="0.00000 0.00016 -0.00000"/>
         <geometry>
           <mesh filename="file://$(find speedy_description)/meshes/dae/Sphere.001.dae" scale="0.35487 0.35487 0.35487"/>
@@ -183,5 +197,5 @@
       </collision>
       <visual name="head">
-        <origin rpy="0.00000 0.00000 0.00000" xyz="0.00000 0.00016 -0.00000"/>
+        <origin rpy="0.00000 ${PI/2} 0.00000" xyz="0.00000 0.00016 -0.00000"/>
         <material name="${white_material}"/>
         <geometry>
@@ -224,4 +238,7 @@
     <color rgba="0.14118 0.14118 0.14118 1.00000"/>
   </material>
+  <material name="grey">
+    <color rgba="0.6 0.6 0.6 1.0000"/>
+  </material>
   <material name="Material.007">
     <color rgba="0.02745 0.02745 0.02745 1.00000"/>

File: speedy_description/urdf/sensors/sensor_camera.urdf.xacro (robot description, xacro)
@@ -3,23 +3,42 @@
 <robot xmlns:xacro="http://wiki.ros.org/xacro">
     <xacro:include filename="$(find speedy_description)/urdf/utils/utils.urdf.xacro"/>
-    <xacro:macro name="sensor_camera" params="prefix parent_link xyz_offset rpy robot_ns">
-        <joint name="${prefix}optical_frame_joint" type="fixed">
+    <xacro:macro name="sensor_camera" params="prefix parent_link xyz_offset rpy robot_ns video_width video_height">
+        <link name="${prefix}camera_frame"/>
+        <joint name="${prefix}camera_joint" type="fixed">
             <origin rpy="${rpy}" xyz="${xyz_offset}"/>
             <parent link="${parent_link}"/>
+            <child link="${prefix}camera_frame"/>
+        </joint>
+        <link name="${prefix}camera_optical_frame"/>
+        <joint name="${prefix}optical_frame_joint" type="fixed">
+            <origin rpy="${-PI/2} 0.00000 ${-PI/2}" xyz="0.00000 0.00000 0.00000"/>
+            <parent link="${prefix}camera_frame"/>
             <child link="${prefix}camera_optical_frame"/>
         </joint>
-        <link name="${prefix}camera_optical_frame">
-            <sensor name="${prefix}camera" type="camera">
-                <origin rpy="-0.00000 -0.00000 -0.00000" xyz="-0.00000 -0.00000 -0.00000"/>
-                <parent link="${prefix}camera_optical_frame"/>
+        <gazebo reference="${prefix}camera_frame">
+            <sensor name="${prefix}sensor" type="camera">
+                <visualize>true</visualize>
+                <update_rate>30</update_rate>
+                <topic>/${robot_ns}/image</topic>
                 <camera>
-                <image>
-                    <width>640</width>
-                    <height>480</height>
-                    <hfov>1.57080</hfov>
-                </image>
+                    <horizontal_fov>${radians(float(90))}</horizontal_fov>
+                    <image>
+                        <width>${video_width}</width>
+                        <height>${video_height}</height>
+                        <format>R8G8B8</format>
+                    </image>
+                    <clip>
+                        <near>0.10</near>
+                        <far>15.0</far>
+                    </clip>
+                    <noise>
+                        <type>gaussian</type>
+                        <mean>0.0</mean>
+                        <stddev>0.007</stddev>
+                    </noise>
+                    <optical_frame_id>${prefix}camera_frame</optical_frame_id>
                 </camera>
             </sensor>
-        </link>
+        </gazebo>
     </xacro:macro>
 </robot>

File: speedy_description/urdf/wheels/rover_wheel.urdf.xacro (robot description, xacro)
@@ -55,4 +55,5 @@
       <origin xyz="${xyz}" rpy="${rpy}"/>
       <axis xyz="${axis_xyz}"/>
+      <limit velocity="1.0" effort="5.0"/>
     </joint>
     <transmission name="${pos}_${side}_wheel_joint_trans">
