Commit message: cmd_vel and all wheels movement working

File: speedy_description/robots/speedy.urdf.xacro (robot description, xacro)
@@ -12,5 +12,5 @@
     <xacro:include filename="$(find speedy_description)/urdf/sensors/sensor_imu.urdf.xacro"/>
     <!-- ARGUMENTS -->
-    <xacro:arg name="robot_ns" default="speedy"/>
+    <xacro:arg name="robot_ns" default=""/>
     <xacro:arg name="prefix" default=""/>
     <xacro:arg name="init_scara_yaw" default="${PI/2}"/>
@@ -37,6 +37,8 @@
     <xacro:property name="bl_wheel_xyz"
                     value="${back_wheel_x_offset} ${wheel_y_offset} ${wheel_z_offset}"/>
-    <xacro:property name="wheels_rpy"
-                    value="${PI/2} 0.00000 0.00000"/>
+    <xacro:property name="right_wheels_rpy"
+                    value="${-PI/2} 0.00000 0.0000"/>
+    <xacro:property name="left_wheels_rpy"
+                    value="${PI/2} 0.00000 0.0000"/>
     <!-- ROBOT PARTS -->
     <!-- base -->
@@ -53,5 +55,5 @@
                         parent_link="$(arg prefix)base_link"
                         xyz="${fr_wheel_xyz}"
-                        rpy="${wheels_rpy}"
+                        rpy="${right_wheels_rpy}"
                         wheel_material="Material.009"
                         prefix="$(arg prefix)"/>
@@ -60,5 +62,5 @@
                         parent_link="$(arg prefix)base_link"
                         xyz="${mr_wheel_xyz}"
-                        rpy="${wheels_rpy}"
+                        rpy="${right_wheels_rpy}"
                         wheel_material="Material.009"
                         prefix="$(arg prefix)"/>
@@ -67,5 +69,5 @@
                         parent_link="$(arg prefix)base_link"
                         xyz="${br_wheel_xyz}"
-                        rpy="${wheels_rpy}"
+                        rpy="${right_wheels_rpy}"
                         wheel_material="Material.009"
                         prefix="$(arg prefix)"/>
@@ -78,5 +80,5 @@
                         parent_link="$(arg prefix)base_link"
                         xyz="${fl_wheel_xyz}"
-                        rpy="${wheels_rpy}"
+                        rpy="${left_wheels_rpy}"
                         wheel_material="Material.009"
                         prefix="$(arg prefix)"/>
@@ -85,5 +87,5 @@
                         parent_link="$(arg prefix)base_link"
                         xyz="${ml_wheel_xyz}"
-                        rpy="${wheels_rpy}"
+                        rpy="${left_wheels_rpy}"
                         wheel_material="Material.009"
                         prefix="$(arg prefix)"/>
@@ -92,5 +94,5 @@
                         parent_link="$(arg prefix)base_link"
                         xyz="${bl_wheel_xyz}"
-                        rpy="${wheels_rpy}"
+                        rpy="${left_wheels_rpy}"
                         wheel_material="Material.009"
                         prefix="$(arg prefix)"/>
@@ -133,5 +135,5 @@
                       rpy="0.00000 0.00000 0.00000"
                       robot_ns="$(arg robot_ns)"
-                      topic="base_imu"/>
+                      topic="base_imu/data"/>
     <!-- GAZEBO ROS2 CONTROL -->
     <xacro:include filename="$(find speedy_description)/urdf/ros2_control.urdf.xacro"/>

File: speedy_description/urdf/arm/gripper.urdf.xacro (robot description, xacro)
@@ -31,5 +31,5 @@
         </link>
         <joint name="${prefix}${side}_gripper_finger_joint" type="prismatic">
-            <limit lower="0.00000" upper="${upper_lim}" effort="0.00000" velocity="0.00000"/>
+            <limit lower="0.00000" upper="${upper_lim}" effort="1000.00000" velocity="100.00000"/>
             <origin rpy="1.57080 0.00000 0.00000" xyz="0.00000 -0.17500 ${offset}"/>
             <parent link="${prefix}${parent_link}"/>

File: speedy_description/urdf/arm/scara.urdf.xacro (robot description, xacro)
@@ -25,5 +25,5 @@
         </link>
         <joint name="${prefix}${name}_joint" type="revolute">
-            <limit lower="${lower_lim}" upper="${upper_lim}" effort="0.00000" velocity="0.00000"/>
+            <limit lower="${lower_lim}" upper="${upper_lim}" effort="1000.00000" velocity="100.00000"/>
             <origin rpy="${rpy}" xyz="${xyz}"/>
             <parent link="${parent_link}"/>
@@ -89,5 +89,5 @@
                 <origin rpy="0.00000 0.00000 0.00000" xyz="-0.00000 0.00000 -0.00000"/>
                 <geometry>
-                    <mesh filename="file://$(find speedy_description)/meshes/dae/Cylinder.024.dae" scale="0.75000 0.75000 1.00000"/>
+                    <mesh filename="package://speedy_description/meshes/dae/Cylinder.024.dae" scale="0.75000 0.75000 1.00000"/>
                 </geometry>
             </collision>
@@ -96,5 +96,5 @@
                 <material name="${white_material}"/>
                 <geometry>
-                    <mesh filename="file://$(find speedy_description)/meshes/dae/Cylinder.024.dae" scale="0.75000 0.75000 1.00000"/>
+                    <mesh filename="package://speedy_description/meshes/dae/Cylinder.024.dae" scale="0.75000 0.75000 1.00000"/>
                 </geometry>
             </visual>
@@ -109,5 +109,5 @@
                 <origin rpy="0.00000 0.00000 0.00000" xyz="0.00000 0.00000 -0.00000"/>
                 <geometry>
-                    <mesh filename="file://$(find speedy_description)/meshes/dae/Cylinder.025.dae" scale="0.43750 0.43750 9.00000"/>
+                    <mesh filename="package://speedy_description/meshes/dae/Cylinder.025.dae" scale="0.43750 0.43750 9.00000"/>
                 </geometry>
             </collision>
@@ -121,5 +121,5 @@
                 <material name="${purple_material}"/>
                 <geometry>
-                    <mesh filename="file://$(find speedy_description)/meshes/dae/Cylinder.025.dae" scale="0.43750 0.43750 9.00000"/>
+                    <mesh filename="package://speedy_description/meshes/dae/Cylinder.025.dae" scale="0.43750 0.43750 9.00000"/>
                 </geometry>
             </visual>
@@ -170,5 +170,5 @@
         </link>
         <joint name="${prefix}scara_prismatic_joint" type="prismatic">
-            <limit lower="-1.30" upper="1.30" effort="0.00000" velocity="0.00000"/>
+            <limit lower="-1.30" upper="1.30" effort="1000.00000" velocity="100.00000"/>
             <origin rpy="0.00000 0.00000 0.00000" xyz="1.00000 -0.00000 -0.00000"/>
             <parent link="${prefix}scara_revolute_arm_2_link"/>
@@ -198,5 +198,5 @@
         </link>
         <joint name="${prefix}scara_wrist_joint" type="revolute">
-            <limit lower="-${PI}" upper="${PI}" effort="0.00000" velocity="0.00000"/>
+            <limit lower="-${PI}" upper="${PI}" effort="1000.00000" velocity="100.00000"/>
             <origin rpy="-${PI} 0.00000 0.00000" xyz="0.00000 0.00000 -1.55000"/>
             <parent link="${prefix}scara_prismatic_link"/>

File: speedy_description/urdf/base/robot_base.urdf.xacro (robot description, xacro)
@@ -133,5 +133,5 @@
         <origin rpy="0.00000 ${PI/2} 0.00000" xyz="0.00000 0.00000 0.00000"/>
         <geometry>
-          <mesh filename="file://$(find speedy_description)/meshes/dae/Cylinder.009.dae" scale="1.00000 1.00000 1.00000"/>
+          <mesh filename="package://speedy_description/meshes/dae/Cylinder.009.dae" scale="1.00000 1.00000 1.00000"/>
         </geometry>
       </collision>
@@ -140,5 +140,5 @@
         <material name="Material.007"/>
         <geometry>
-          <mesh filename="file://$(find speedy_description)/meshes/dae/Cylinder.009.dae" scale="1.00000 1.00000 1.00000"/>
+          <mesh filename="package://speedy_description/meshes/dae/Cylinder.009.dae" scale="1.00000 1.00000 1.00000"/>
         </geometry>
       </visual>
@@ -173,5 +173,5 @@
         <origin rpy="0.00000 ${PI/2} 0.00000" xyz="0.00000 -0.00000 -0.00000"/>
         <geometry>
-          <mesh filename="file://$(find speedy_description)/meshes/dae/Cylinder.004.dae" scale="0.35487 0.35487 0.44358"/>
+          <mesh filename="package://speedy_description/meshes/dae/Cylinder.004.dae" scale="0.35487 0.35487 0.44358"/>
         </geometry>
       </collision>
@@ -180,5 +180,5 @@
         <material name="Material.005"/>
         <geometry>
-          <mesh filename="file://$(find speedy_description)/meshes/dae/Cylinder.004.dae" scale="0.35487 0.35487 0.44358"/>
+          <mesh filename="package://speedy_description/meshes/dae/Cylinder.004.dae" scale="0.35487 0.35487 0.44358"/>
         </geometry>
       </visual>
@@ -193,5 +193,5 @@
         <origin rpy="0.00000 ${PI/2} 0.00000" xyz="0.00000 0.00016 -0.00000"/>
         <geometry>
-          <mesh filename="file://$(find speedy_description)/meshes/dae/Sphere.001.dae" scale="0.35487 0.35487 0.35487"/>
+          <mesh filename="package://speedy_description/meshes/dae/Sphere.001.dae" scale="0.35487 0.35487 0.35487"/>
         </geometry>
       </collision>
@@ -200,5 +200,5 @@
         <material name="${white_material}"/>
         <geometry>
-          <mesh filename="file://$(find speedy_description)/meshes/dae/Sphere.001.dae" scale="0.35487 0.35487 0.35487"/>
+          <mesh filename="package://speedy_description/meshes/dae/Sphere.001.dae" scale="0.35487 0.35487 0.35487"/>
         </geometry>
       </visual>
@@ -213,5 +213,5 @@
         <origin rpy="0.00000 0.00000 0.00000" xyz="0.00000 -0.00016 -0.00000"/>
         <geometry>
-          <mesh filename="file://$(find speedy_description)/meshes/dae/Cylinder.007.dae" scale="0.70974 0.70974 0.70974"/>
+          <mesh filename="package://speedy_description/meshes/dae/Cylinder.007.dae" scale="0.70974 0.70974 0.70974"/>
         </geometry>
       </collision>
@@ -225,5 +225,5 @@
         <material name="${white_material}"/>
         <geometry>
-          <mesh filename="file://$(find speedy_description)/meshes/dae/Cylinder.007.dae" scale="0.70974 0.70974 0.70974"/>
+          <mesh filename="package://speedy_description/meshes/dae/Cylinder.007.dae" scale="0.70974 0.70974 0.70974"/>
         </geometry>
       </visual>

File: speedy_description/urdf/ros2_control.urdf.xacro (robot description, xacro)
@@ -13,6 +13,6 @@
             <joint name="${frame_prefix}front_left_wheel_joint">
                 <command_interface name="velocity">
-                    <param name="min">-1</param>
-                    <param name="max">1</param>
+                    <param name="min">-5.1282</param>
+                    <param name="max">5.1282</param>
                 </command_interface>
                 <state_interface name="position"/>
@@ -22,6 +22,6 @@
             <joint name="${frame_prefix}front_right_wheel_joint">
                 <command_interface name="velocity">
-                    <param name="min">-1</param>
-                    <param name="max">1</param>
+                    <param name="min">-5.1282</param>
+                    <param name="max">5.1282</param>
                 </command_interface>
                 <state_interface name="position"/>
@@ -31,6 +31,6 @@
             <joint name="${frame_prefix}back_right_wheel_joint">
                 <command_interface name="velocity">
-                    <param name="min">-1</param>
-                    <param name="max">1</param>
+                    <param name="min">-5.1282</param>
+                    <param name="max">5.1282</param>
                 </command_interface>
                 <state_interface name="position"/>
@@ -40,6 +40,6 @@
             <joint name="${frame_prefix}back_left_wheel_joint">
                 <command_interface name="velocity">
-                    <param name="min">-1</param>
-                    <param name="max">1</param>
+                    <param name="min">-5.1282</param>
+                    <param name="max">5.1282</param>
                 </command_interface>
                 <state_interface name="position"/>
@@ -49,6 +49,6 @@
             <joint name="${frame_prefix}mid_right_wheel_joint">
                 <command_interface name="velocity">
-                    <param name="min">-1</param>
-                    <param name="max">1</param>
+                    <param name="min">-5.1282</param>
+                    <param name="max">5.1282</param>
                 </command_interface>
                 <state_interface name="position"/>
@@ -58,6 +58,6 @@
             <joint name="${frame_prefix}mid_left_wheel_joint">
                 <command_interface name="velocity">
-                    <param name="min">-1</param>
-                    <param name="max">1</param>
+                    <param name="min">-5.1282</param>
+                    <param name="max">5.1282</param>
                 </command_interface>
                 <state_interface name="position"/>

File: speedy_description/urdf/sensors/sensor_camera.urdf.xacro (robot description, xacro)
@@ -20,5 +20,5 @@
                 <visualize>true</visualize>
                 <update_rate>30</update_rate>
-                <topic>/${robot_ns}/image</topic>
+                <topic>${robot_ns}/${prefix}camera/image</topic>
                 <camera>
                     <horizontal_fov>${radians(float(90))}</horizontal_fov>

File: speedy_description/urdf/sensors/sensor_imu.urdf.xacro (robot description, xacro)
@@ -9,7 +9,7 @@
             <child link="${prefix}imu_sensor_link"/>
         </joint>
-        <link name="${prefix}imu_sensor_link">
-            <gazebo reference="${prefix}imu_sensor_link">
-            <sensor name="${prefix}_sensor" type="imu">
+        <link name="${prefix}imu_sensor_link"/>
+        <gazebo reference="${prefix}imu_sensor_link">
+            <sensor name="${prefix}sensor" type="imu">
                 <always_on>1</always_on>
                 <update_rate>30</update_rate>
@@ -17,5 +17,4 @@
             </sensor>
         </gazebo>
-        </link>
     </xacro:macro>
 </robot>

File: speedy_description/urdf/wheels/rover_wheel.urdf.xacro (robot description, xacro)
@@ -3,13 +3,4 @@
 <robot xmlns:xacro="http://wiki.ros.org/xacro">
   <xacro:macro name="rover_wheel" params="side pos parent_link xyz rpy wheel_material prefix">
-    <!--
-      rover_wheel
-      PARAMS
-        · side: right/left
-        · pos: front/mid/back
-        · parent_link: name of parent link
-        · xyz: x,y,z position of the wheel
-        · rpy: x,y,z rotation of the wheel
-    -->
     <xacro:if value="${side != 'left' and side != 'right'}">
       <xacro:error message="'side' parameter must be 'right' or 'left'."/>
@@ -18,16 +9,15 @@
       <xacro:error message="'pos' parameter must be 'front', 'mid' or 'back'."/>
     </xacro:if>
-    <xacro:property name="axis_xyz" value="0.00000 0.00000 -1.00000"/>
     <link name="${pos}_${side}_wheel_link">
       <collision name="${pos}_${side}_wheel_collision">
         <origin rpy="0.00000 -0.00000 -0.00000" xyz="-0.00000 -0.00000 -0.00000"/>
         <geometry>
-          <mesh filename="file://$(find speedy_description)/meshes/dae/Torus.001.dae" scale="0.66102 0.66102 0.58333"/>
+          <mesh filename="package://speedy_description/meshes/dae/Torus.001.dae" scale="0.66102 0.66102 0.58333"/>
         </geometry>
         <surface>
           <friction>
             <ode>
-              <mu>1.000000</mu>
-              <mu2>1.000000</mu2>
+              <mu>20.000000</mu>
+              <mu2>20.000000</mu2>
               <fdir1>0.0000 0.0000 1.0000</fdir1>
               <slip1>0.50000</slip1>
@@ -46,5 +36,5 @@
         <material name="${wheel_material}"/>
         <geometry>
-          <mesh filename="file://$(find speedy_description)/meshes/dae/Torus.001.dae" scale="0.66102 0.66102 0.58333"/>
+          <mesh filename="package://speedy_description/meshes/dae/Torus.001.dae" scale="0.66102 0.66102 0.58333"/>
         </geometry>
       </visual>
@@ -54,14 +44,14 @@
       <child link="${pos}_${side}_wheel_link"/>
       <origin xyz="${xyz}" rpy="${rpy}"/>
-      <axis xyz="${axis_xyz}"/>
-      <limit velocity="1.0" effort="5.0"/>
+      <axis xyz="0.00000 0.00000 1.00000"/>
+      <limit velocity="5.1282" effort="1000.0"/>
     </joint>
     <transmission name="${pos}_${side}_wheel_joint_trans">
       <type>transmission_interface/SimpleTransmission</type>
       <joint name="${pos}_${side}_wheel_joint">
-        <hardwareInterface>hardware_interface/PositionJointInterface</hardwareInterface>
+        <hardwareInterface>hardware_interface/VelocityJointInterface</hardwareInterface>
       </joint>
       <actuator name="${pos}_${side}_wheel_joint_motor">
-        <mechanicalReduction></mechanicalReduction>
+        <mechanicalReduction>1</mechanicalReduction>
       </actuator>
     </transmission>
@@ -69,4 +59,8 @@
       <mu1>5</mu1>
       <mu2>5</mu2>
+      <kp>2.72e6</kp>
+      <kd>8.25e1</kd>
+      <fdir1>0 0 0</fdir1>
+      <maxContacts>4</maxContacts>
     </gazebo>
   </xacro:macro>
