Commit message: cmd_vel and all wheels movement working

File: speedy_description/urdf/wheels/wheels_chasis.urdf.xacro (robot description, xacro)
@@ -18,5 +18,5 @@
         <origin rpy="-0.00000 -0.00000 -0.00000" xyz="-0.00000 0.00000 -0.00000"/>
         <geometry>
-          <mesh filename="file://$(find speedy_description)/meshes/dae/Cube.018.dae" scale="0.10000 0.04007 0.30000"/>
+          <mesh filename="package://speedy_description/meshes/dae/Cube.018.dae" scale="0.10000 0.04007 0.30000"/>
         </geometry>
       </collision>
@@ -44,5 +44,5 @@
         <origin rpy="-0.00000 0.00000 0.00000" xyz="-0.00000 -0.00000 -0.00000"/>
         <geometry>
-          <mesh filename="file://$(find speedy_description)/meshes/dae/Cube.003.dae" scale="0.10000 0.26800 0.03775"/>
+          <mesh filename="package://speedy_description/meshes/dae/Cube.003.dae" scale="0.10000 0.26800 0.03775"/>
         </geometry>
       </collision>
@@ -70,5 +70,5 @@
         <origin rpy="${PI/2} -0.00000 -0.00000" xyz="-0.00000 0.00000 -0.00000"/>
         <geometry>
-          <mesh filename="file://$(find speedy_description)/meshes/dae/Cylinder.003.dae" scale="0.70000 0.70000 2.00000"/>
+          <mesh filename="package://speedy_description/meshes/dae/Cylinder.003.dae" scale="0.70000 0.70000 2.00000"/>
         </geometry>
       </collision>
@@ -81,5 +81,5 @@
         <origin rpy="${PI/2} -0.00000 0.00000" xyz="-0.00000 0.00000 -0.00000"/>
         <geometry>
-          <mesh filename="file://$(find speedy_description)/meshes/dae/Cylinder.003.dae" scale="0.70000 0.70000 2.00000"/>
+          <mesh filename="package://speedy_description/meshes/dae/Cylinder.003.dae" scale="0.70000 0.70000 2.00000"/>
         </geometry>
       </visual>
@@ -108,5 +108,5 @@
         <origin rpy="-0.00000 0.00000 0.00000" xyz="0.00000 -0.00000 0.00000"/>
         <geometry>
-          <mesh filename="file://$(find speedy_description)/meshes/dae/Cylinder.022.dae" scale="1.00000 1.00000 1.92308"/>
+          <mesh filename="package://speedy_description/meshes/dae/Cylinder.022.dae" scale="1.00000 1.00000 1.92308"/>
         </geometry>
       </collision>
@@ -120,5 +120,5 @@
         <material name="Material.016"/>
         <geometry>
-          <mesh filename="file://$(find speedy_description)/meshes/dae/Cylinder.022.dae" scale="1.00000 1.00000 1.92308"/>
+          <mesh filename="package://speedy_description/meshes/dae/Cylinder.022.dae" scale="1.00000 1.00000 1.92308"/>
         </geometry>
       </visual>
@@ -133,5 +133,5 @@
         <origin rpy="-0.00000 0.00000 0.00000" xyz="0.00000 0.00000 -0.00000"/>
         <geometry>
-          <mesh filename="file://$(find speedy_description)/meshes/dae/Sphere.006.dae" scale="1.00000 1.00000 1.00000"/>
+          <mesh filename="package://speedy_description/meshes/dae/Sphere.006.dae" scale="1.00000 1.00000 1.00000"/>
         </geometry>
       </collision>
@@ -145,5 +145,5 @@
         <material name="Material.016"/>
         <geometry>
-          <mesh filename="file://$(find speedy_description)/meshes/dae/Sphere.006.dae" scale="1.00000 1.00000 1.00000"/>
+          <mesh filename="package://speedy_description/meshes/dae/Sphere.006.dae" scale="1.00000 1.00000 1.00000"/>
         </geometry>
       </visual>
@@ -158,5 +158,5 @@
         <origin rpy="0.00000 -0.00000 -0.00000" xyz="-0.00000 0.00000 0.00000"/>
         <geometry>
-          <mesh filename="file://$(find speedy_description)/meshes/dae/Cylinder.dae" scale="0.05000 0.05000 0.38165"/>
+          <mesh filename="package://speedy_description/meshes/dae/Cylinder.dae" scale="0.05000 0.05000 0.38165"/>
         </geometry>
       </collision>
@@ -170,5 +170,5 @@
         <material name="Material"/>
         <geometry>
-          <mesh filename="file://$(find speedy_description)/meshes/dae/Cylinder.dae" scale="0.05000 0.05000 0.38165"/>
+          <mesh filename="package://speedy_description/meshes/dae/Cylinder.dae" scale="0.05000 0.05000 0.38165"/>
         </geometry>
       </visual>
@@ -183,5 +183,5 @@
         <origin rpy="-0.00000 0.00000 0.00000" xyz="-0.00000 0.00000 0.00000"/>
         <geometry>
-          <mesh filename="file://$(find speedy_description)/meshes/dae/Sphere.dae" scale="0.08862 0.08862 0.08862"/>
+          <mesh filename="package://speedy_description/meshes/dae/Sphere.dae" scale="0.08862 0.08862 0.08862"/>
         </geometry>
       </collision>
@@ -195,5 +195,5 @@
         <material name="Material.002"/>
         <geometry>
-          <mesh filename="file://$(find speedy_description)/meshes/dae/Sphere.dae" scale="0.08862 0.08862 0.08862"/>
+          <mesh filename="package://speedy_description/meshes/dae/Sphere.dae" scale="0.08862 0.08862 0.08862"/>
         </geometry>
       </visual>
@@ -210,5 +210,5 @@
         <origin rpy="-0.00000 -0.00000 -0.00000" xyz="-0.00000 -0.00000 -0.00000"/>
         <geometry>
-          <mesh filename="file://$(find speedy_description)/meshes/dae/Cylinder.006.dae" scale="0.05000 0.05000 0.39665"/>
+          <mesh filename="package://speedy_description/meshes/dae/Cylinder.006.dae" scale="0.05000 0.05000 0.39665"/>
         </geometry>
       </collision>
@@ -222,5 +222,5 @@
         <material name="Material"/>
         <geometry>
-          <mesh filename="file://$(find speedy_description)/meshes/dae/Cylinder.006.dae" scale="0.05000 0.05000 0.39665"/>
+          <mesh filename="package://speedy_description/meshes/dae/Cylinder.006.dae" scale="0.05000 0.05000 0.39665"/>
         </geometry>
       </visual>
@@ -242,5 +242,5 @@
         <origin rpy="-0.00000 -0.00000 0.00000" xyz="-0.00000 -0.00000 -0.00000"/>
         <geometry>
-          <mesh filename="file://$(find speedy_description)/meshes/dae/Cylinder.019.dae" scale="0.83333 0.83333 11.25616"/>
+          <mesh filename="package://speedy_description/meshes/dae/Cylinder.019.dae" scale="0.83333 0.83333 11.25616"/>
         </geometry>
       </collision>
@@ -254,5 +254,5 @@
         <material name="Material.010"/>
         <geometry>
-          <mesh filename="file://$(find speedy_description)/meshes/dae/Cylinder.019.dae" scale="0.83333 0.83333 11.25615"/>
+          <mesh filename="package://speedy_description/meshes/dae/Cylinder.019.dae" scale="0.83333 0.83333 11.25615"/>
         </geometry>
       </visual>
@@ -274,5 +274,5 @@
         <origin rpy="-0.00000 0.00000 0.00000" xyz="0.00000 -0.00000 0.00000"/>
         <geometry>
-          <mesh filename="file://$(find speedy_description)/meshes/dae/Cylinder.008.dae" scale="0.05000 0.05000 0.38165"/>
+          <mesh filename="package://speedy_description/meshes/dae/Cylinder.008.dae" scale="0.05000 0.05000 0.38165"/>
         </geometry>
       </collision>
@@ -286,5 +286,5 @@
         <material name="Material"/>
         <geometry>
-          <mesh filename="file://$(find speedy_description)/meshes/dae/Cylinder.008.dae" scale="0.05000 0.05000 0.38165"/>
+          <mesh filename="package://speedy_description/meshes/dae/Cylinder.008.dae" scale="0.05000 0.05000 0.38165"/>
         </geometry>
       </visual>
